File: hw/bldc/bldc.kicad_pcb (KiCad board)
At the start: 2 copper layers, 54 x 29.2 mm, 71 parts, among them IC1 MP2315SGJ-P, J1 Conn_01x05, J3 Conn_01x06, Q1 BSC13DN30NSFD, Q10 BSC13DN30NSFD, Q2 BSC13DN30NSFD, Q7 BSC13DN30NSFD, Q8 BSC13DN30NSFD, Q9 BSC13DN30NSFD, U1 LD1117S33TR_SOT223, U2 IR2101, U3 IR2101, U4 IR2101, U5 STM32L431CCTx

Commit message: pcb update
Parts:
- added TP10: C, TestPoint:TestPoint_Pad_D1.0mm, F.Cu at (65.2, 111.5)
- added TP11: C, TestPoint:TestPoint_Pad_D1.0mm, F.Cu at (66.5, 109.0)
Connections:
- U5 pad 25: unconnected-(U5-PB12-Pad25) -> Net-(U5-PB12)
- U5 pad 27: unconnected-(U5-PB14-Pad27) -> Net-(U5-PB14)
Routing:
- net Net-(U5-PB14): track 0.00 -> 2.09 mm
- net Net-(U5-PB12): track 0.00 -> 1.85 mm
Other:
- board text added: "BEMF"
- board text added: "BLDC Driver"
- board text added: "VIN"
- board text added: "mayankpatel468@gmail.com"
- board text removed: "TO DO ================================= * Label each and every pad * check inductor pad, mosfet pad * Place mosfets at the bottom, for heatsink * keep all the solderpads at TOP"
