File: hw/bldc/bldc.kicad_pcb (KiCad board)
At the start: 2 copper layers, 54 x 29.2 mm, 73 parts, among them IC1 MP2315SGJ-P, J1 Conn_01x05, J3 Conn_01x06, Q1 BSC13DN30NSFD, Q10 BSC13DN30NSFD, Q2 BSC13DN30NSFD, Q7 BSC13DN30NSFD, Q8 BSC13DN30NSFD, Q9 BSC13DN30NSFD, U1 LD1117S33TR_SOT223, U2 IR2101, U3 IR2101, U4 IR2101, U5 STM32L431CCTx

Commit message: made some corrections
Parts:
- added TP12: C, TestPoint:TestPoint_Pad_D1.0mm, F.Cu at (67.2, 106.0)
- moved TP11 5.10 mm to (67.5, 104.0)
- moved C11 0.50 mm to (65.8, 102.2)
- moved R4 0.50 mm to (87.0, 110.8)
Connections:
- TP11 pad 1: Net-(U5-PB14) -> Net-(U5-PA12)
- U5 pad 27: Net-(U5-PB14) -> /RPM
- U5 pad 32: /LED -> Net-(U5-PA11)
- U5 pad 33: unconnected-(U5-PA12-Pad33) -> Net-(U5-PA12)
- U5 pad 41: unconnected-(U5-PB5-Pad41) -> /LED
Routing:
- net /LED: track 15.4 -> 6.83 mm, vias 0 -> 2
- net /RPM: track 0.00 -> 5.06 mm, vias 0 -> 1
- net Net-(U5-PA12): track 0.00 -> 3.92 mm
- net Net-(U5-PA11): track 0.00 -> 3.04 mm
- net GND: track 81.9 -> 84.5 mm, vias 22 -> 24
- net Net-(U5-PB14): track 2.09 -> 0.00 mm
- net +3V3: track 69.6 -> 68.9 mm
- net Net-(Q8-G): track 2.63 -> 2.09 mm
- net Net-(U3-LO): track 2.45 -> 2.95 mm
Other:
- board text added: "PA11"
- board text added: "PA12"
- board text added: "PB12"
