File: hw/bldc/bldc.kicad_sch (KiCad schematic)
At the start: 73 parts, among them IC1 MP2315SGJ-P, J1 Conn_01x05, J3 Conn_01x06, Q1 BSC13DN30NSFD, Q10 BSC13DN30NSFD, Q2 BSC13DN30NSFD, Q7 BSC13DN30NSFD, Q8 BSC13DN30NSFD, Q9 BSC13DN30NSFD, U1 LD1117S33TR_SOT223, U2 IR2101, U3 IR2101, U4 IR2101, U5 STM32L431CCTx

Commit message: made some corrections
Parts:
- added TP12: C, TestPoint:TestPoint_Pad_D1.0mm, symbol Connector:TestPoint
Connections:
- net LED: now also U5.41 (PB5); no longer U5.32 (PA11)
- net RPM: now also U5.27 (PB14)
- net at TP11.1: now also U5.33 (PA12); no longer U5.27 (PB14)
- new net: TP12.1, U5.32 (PA11)
Changed lines of the file:
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@@
 	(wire
 		(pts
+			(xy 19.05 151.13) (xy 30.48 151.13)
+		)
+		(stroke
+			(width 0)
+			(type default)
+		)
+	)
+	(wire
+		(pts
 			(xy 177.8 149.86) (xy 177.8 152.4)
 		)
@@
 	(wire
 		(pts
-			(xy 27.94 173.99) (xy 30.48 173.99)
+			(xy 24.13 173.99) (xy 30.48 173.99)
 		)
 		(stroke
@@
 	(wire
 		(pts
-			(xy 48.26 104.14) (xy 50.8 104.14)
+			(xy 72.39 143.51) (xy 60.96 143.51)
 		)
 		(stroke
@@
 	(wire
 		(pts
-			(xy 246.38 114.3) (xy 252.73 114.3)
+			(xy 48.26 104.14) (xy 50.8 104.14)
 		)
 		(stroke
@@
 	(wire
 		(pts
-			(xy 40.64 107.95) (xy 40.64 104.14)
+			(xy 246.38 114.3) (xy 252.73 114.3)
 		)
 		(stroke
@@
 	(wire
 		(pts
-			(xy 45.72 104.14) (xy 48.26 104.14)
+			(xy 40.64 107.95) (xy 40.64 104.14)
 		)
 		(stroke
@@
 	(wire
 		(pts
-			(xy 158.75 88.9) (xy 170.18 88.9)
+			(xy 45.72 104.14) (xy 48.26 104.14)
 		)
 		(stroke
@@
 	(wire
 		(pts
-			(xy 67.31 140.97) (xy 60.96 140.97)
+			(xy 158.75 88.9) (xy 170.18 88.9)
 		)
 		(stroke
@@
 	(wire
 		(pts
+			(xy 72.39 140.97) (xy 60.96 140.97)
+		)
+		(stroke
+			(width 0)
+			(type default)
+		)
+	)
+	(wire
+		(pts
 			(xy 250.19 49.53) (xy 255.27 49.53)
 		)
@@
 		)
 	)
-	(label "FB"
-		(at 76.2 36.83 0)
+	(label "LED"
+		(at 19.05 151.13 0)
 		(fields_autoplaced yes)
 		(effects
@@
 		)
 	)
-	(label "TIM1_CH3N"
-		(at 158.75 40.64 0)
+	(label "FB"
+		(at 76.2 36.83 0)
 		(fields_autoplaced yes)
 		(effects
@@
 		)
 	)
-	(label "SWDIO"
-		(at 114.3 181.61 180)
+	(label "TIM1_CH3N"
+		(at 158.75 40.64 0)
 		(fields_autoplaced yes)
 		(effects
@@
 				(size 1.27 1.27)
 			)
-			(justify right bottom)
+			(justify left bottom)
 		)
 	)
-	(label "LED"
-		(at 67.31 140.97 180)
+	(label "SWDIO"
+		(at 114.3 181.61 180)
 		(fields_autoplaced yes)
 		(effects
@@
 		)
 	)
+	(label "RPM"
+		(at 24.13 173.99 0)
+		(fields_autoplaced yes)
+		(effects
+			(font
+				(size 1.27 1.27)
+			)
+			(justify left bottom)
+		)
+	)
 	(label "TIM1_CH2N"
 		(at 19.05 138.43 0)
@@
 	(symbol
 		(lib_id "Connector:TestPoint")
-		(at 27.94 173.99 90)
+		(at 29.21 73.66 90)
 		(unit 1)
 		(exclude_from_sim no)
@@
 		(on_board yes)
 		(dnp no)
-		(property "Reference" "TP11"
-			(at 22.86 175.2601 90)
+		(property "Reference" "TP9"
+			(at 22.86 73.914 90)
 			(effects
 				(font
 					(size 1.27 1.27)
 				)
-				(justify left)
 			)
 		)
-		(property "Value" "C"
-			(at 22.86 172.7201 90)
+		(property "Value" "SP"
+			(at 18.796 73.66 90)
 			(effects
 				(font
 					(size 1.27 1.27)
 				)
-				(justify left)
 			)
 		)
-		(property "Footprint" "TestPoint:TestPoint_Pad_D1.0mm"
-			(at 27.94 168.91 0)
+		(property "Footprint" "TestPoint:TestPoint_Pad_3.0x3.0mm"
+			(at 29.21 68.58 0)
 			(effects
 				(font
@@
 		)
 		(property "Datasheet" "~"
-			(at 27.94 168.91 0)
+			(at 29.21 68.58 0)
 			(effects
 				(font
@@
 		)
 		(property "Description" "test point"
-			(at 27.94 173.99 0)
+			(at 29.21 73.66 0)
 			(effects
 				(font
@@
 			(project "bldc"
 				(path "/8f50835c-fbe0-401c-8ea4-1e9972c1e8f7"
-					(reference "TP11")
+					(reference "TP9")
 					(unit 1)
 				)
@@
 	(symbol
 		(lib_id "Connector:TestPoint")
-		(at 29.21 73.66 90)
+		(at 72.39 140.97 270)
 		(unit 1)
 		(exclude_from_sim no)
@@
 		(on_board yes)
 		(dnp no)
-		(property "Reference" "TP9"
-			(at 22.86 73.914 90)
+		(property "Reference" "TP12"
+			(at 76.962 140.97 90)
 			(effects
 				(font
 					(size 1.27 1.27)
 				)
+				(justify left)
 			)
 		)
-		(property "Value" "SP"
-			(at 18.796 73.66 90)
+		(property "Value" "C"
+			(at 85.598 140.97 90)
 			(effects
 				(font
 					(size 1.27 1.27)
 				)
+				(justify left)
 			)
 		)
-		(property "Footprint" "TestPoint:TestPoint_Pad_3.0x3.0mm"
-			(at 29.21 68.58 0)
+		(property "Footprint" "TestPoint:TestPoint_Pad_D1.0mm"
+			(at 72.39 146.05 0)
 			(effects
 				(font
@@
 		)
 		(property "Datasheet" "~"
-			(at 29.21 68.58 0)
+			(at 72.39 146.05 0)
 			(effects
 				(font
@@
 		)
 		(property "Description" "test point"
-			(at 29.21 73.66 0)
+			(at 72.39 140.97 0)
 			(effects
 				(font
@@
 			(project "bldc"
 				(path "/8f50835c-fbe0-401c-8ea4-1e9972c1e8f7"
-					(reference "TP9")
+					(reference "TP12")
 					(unit 1)
 				)
@@
 					(unit 1)
 				)
+			)
+		)
+	)
+	(symbol
+		(lib_id "Connector:TestPoint")
+		(at 72.39 143.51 270)
+		(unit 1)
+		(exclude_from_sim no)
+		(in_bom yes)
+		(on_board yes)
+		(dnp no)
+		(property "Reference" "TP11"
+			(at 76.962 143.764 90)
+			(effects
+				(font
+					(size 1.27 1.27)
+				)
+				(justify left)
+			)
+		)
+		(property "Value" "C"
+			(at 85.598 143.764 90)
+			(effects
+				(font
+					(size 1.27 1.27)
+				)
+				(justify left)
+			)
+		)
+		(property "Footprint" "TestPoint:TestPoint_Pad_D1.0mm"
+			(at 72.39 148.59 0)
+			(effects
+				(font
+					(size 1.27 1.27)
+				)
+				(hide yes)
+			)
+		)
+		(property "Datasheet" "~"
+			(at 72.39 148.59 0)
+			(effects
+				(font
+					(size 1.27 1.27)
+				)
+				(hide yes)
+			)
+		)
+		(property "Description" "test point"
+			(at 72.39 143.51 0)
+			(effects
+				(font
+					(size 1.27 1.27)
+				)
+				(hide yes)
+			)
+		)
+		(pin "1"
+		)
+		(instances
+			(project "bldc"
+				(path "/8f50835c-fbe0-401c-8ea4-1e9972c1e8f7"
+					(reference "TP11")
+					(unit 1)
+				)
